File: hardware/Digital-Input.kicad_sch (KiCad schematic)
At the start: 0 parts

Commit message: Layout updates
Signed-off-by: Connor Rigby <connorr@hey.com>
Parts:
- added C701, C702, C703, C704: C_0603_DNP, Capacitor_SMD:C_0603_1608Metric, symbol LCSC_Capacitor:C_0603_DNP
- added R701, R702, R703, R704, R705, R706, R707, R708: DNP, Resistor_SMD:R_0603_1608Metric, symbol LCSC_Resistor:R_0603_DNP
Connections:
- net DI_1: now also R707.1
- net DI_1_TTL: now also C701.1, R701.2, R702.2
- net DI_2: now also R705.1
- net DI_2_TTL: now also C702.1, R703.2, R704.2
- net DI_3: now also R703.1
- net DI_3_TTL: now also C703.1, R705.2, R706.2
- net DI_4: now also R701.1
- net DI_4_TTL: now also C704.1, R707.2, R708.2
- new net GND: C701.2, C702.2, C703.2, C704.2, R702.1, R704.1, R706.1, R708.1

Commit message: Almost ready for fab
Signed-off-by: Connor Rigby <connorr@hey.com>
Parts:
- removed R701, R702, R703, R704, R705, R706, R707, R708: DNP, Resistor_SMD:R_0603_1608Metric, symbol LCSC_Resistor:R_0603_DNP
- added R701, R703, R705, R707: R_0603_100k, Resistor_SMD:R_0603_1608Metric, symbol LCSC_Resistor:R_0603_100k
- added R702, R704, R706, R708: R_0603_20k, Resistor_SMD:R_0603_1608Metric, symbol LCSC_Resistor:R_0603_20k
- C701, C702, C703, C704: now not fitted
Connections:
- net DI_1: now also R707.1
- net DI_1_TTL: now also R701.2, R702.2
- net DI_2: now also R705.1
- net DI_2_TTL: now also R703.2, R704.2
- net DI_3: now also R703.1
- net DI_3_TTL: now also R705.2, R706.2
- net DI_4: now also R701.1
- net DI_4_TTL: now also R707.2, R708.2
- net GND: now also R702.1, R704.1, R706.1, R708.1
Other:
- note added: "(V_{s} x R_{2}Ω) / (R_{1}Ω + R_{2}Ω) = V_{out} V_{s} = 12 | R_{1} = 100kΩ | R_{2} = 20kΩ @ 10v = 1.7V (low) @ 12v = 2V (nominal) @ 20v = 3.~{33} (high)"

Commit message: Pre-production updates
Signed-off-by: Connor Rigby <connorr@hey.com>
Other:
- company: (none) -> https://cone.codes
- title: (none) -> coneRGB2
Changed lines of the file:
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@@
 (kicad_sch (version 20230121) (generator eeschema)
   (paper "A5")
+  (title_block
+    (title "coneRGB2")
+    (date "2023-03-20")
+    (rev "1")
+    (company "https://cone.codes")
+    (comment 1 "https://github.com/connorrigby/underglow2")
+    (comment 2 "Designed by Connor Rigby")
+    (comment 3 "Steps between 10 and 20 volts down to a save 3.3v for the MCU")
+    (comment 4 "Digital External 12v Input")
+  )
   (junction (at 121.92 67.31) (diameter 0) (color 0 0 0 0)
   )
@@
     (stroke (width 0) (type default))
   )
+  (text_box "Simple resistor divider to prevent excess voltage and current from entering the MCU's GPIO pins.\nCapacitors placed but not populated in case future installs need debouncing\nor additional filtering"
+    (at 76.2 85.09 0) (size 53.34 11.43)
+    (stroke (width 0) (type default))
+    (fill (type none))
+    (effects (font (size 1.27 1.27)) (justify left top))
+  )
   (text "(V_{s} x R_{2}Ω) / (R_{1}Ω + R_{2}Ω) = V_{out}\nV_{s} = 12 | R_{1} = 100kΩ | R_{2} = 20kΩ\n\n@ 10v = 1.7V (low)\n\n@ 12v = 2V (nominal)\n\n@ 20v = 3.~{33} (high)"

Commit message: Rev 2 submitted for production
Signed-off-by: Connor Rigby <connorr@hey.com>
Connections:
- net DI_1: now also R701.1; no longer R707.1
- net DI_2: now also R703.1; no longer R705.1
- net DI_3: now also R705.1; no longer R703.1
- net DI_4: now also R707.1; no longer R701.1
- net DI_1_TTL renamed PI1
- net DI_2_TTL renamed PI2
- net DI_3_TTL renamed PI3
- net DI_4_TTL renamed PI4
Changed lines of the file:
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@@
   (title_block
     (title "coneRGB2")
-    (date "2023-03-20")
-    (rev "1")
+    (date "2023-05-04")
+    (rev "2")
     (company "https://cone.codes")
     (comment 1 "https://github.com/connorrigby/underglow2")
@@
     (effects (font (size 1.27 1.27)) (justify left bottom))
   )
-  (hierarchical_label "DI_2_TTL" (shape output) (at 81.28 63.5 90) (fields_autoplaced)
+  (hierarchical_label "PI3" (shape output) (at 101.6 63.5 90) (fields_autoplaced)
+    (effects (font (size 1.27 1.27)) (justify left))
+    (property "Netclass" "GPIO" (at 105.41 63.5 90)
+      (effects (font (size 1.27 1.27) italic) (justify left) hide)
+    )
+  )
+  (hierarchical_label "PI2" (shape output) (at 81.28 63.5 90) (fields_autoplaced)
+    (effects (font (size 1.27 1.27)) (justify left))
+    (property "Netclass" "GPIO" (at 85.09 63.5 90)
+      (effects (font (size 1.27 1.27) italic) (justify left) hide)
+    )
+  )
+  (hierarchical_label "DI_1" (shape input) (at 53.34 46.99 90) (fields_autoplaced)
     (effects (font (size 1.27 1.27)) (justify left))
   )
-  (hierarchical_label "DI_1" (shape input) (at 116.84 46.99 90) (fields_autoplaced)
+  (hierarchical_label "PI4" (shape output) (at 121.92 63.5 90) (fields_autoplaced)
+    (effects (font (size 1.27 1.27)) (justify left))
+    (property "Netclass" "GPIO" (at 120.65 63.5 90)
+      (effects (font (size 1.27 1.27) italic) (justify left) hide)
+    )
+  )
+  (hierarchical_label "DI_3" (shape input) (at 96.52 46.99 90) (fields_autoplaced)
     (effects (font (size 1.27 1.27)) (justify left))
   )
-  (hierarchical_label "DI_4_TTL" (shape output) (at 121.92 63.5 90) (fields_autoplaced)
+  (hierarchical_label "PI1" (shape output) (at 58.42 63.5 90) (fields_autoplaced)
+    (effects (font (size 1.27 1.27)) (justify left))
+    (property "Netclass" "GPIO" (at 57.15 63.5 90)
+      (effects (font (size 1.27 1.27) italic) (justify left) hide)
+    )
+  )
+  (hierarchical_label "DI_4" (shape input) (at 116.84 46.99 90) (fields_autoplaced)
     (effects (font (size 1.27 1.27)) (justify left))
   )
-  (hierarchical_label "DI_1_TTL" (shape output) (at 58.42 63.5 90) (fields_autoplaced)
+  (hierarchical_label "DI_2" (shape input) (at 76.2 46.99 90) (fields_autoplaced)
     (effects (font (size 1.27 1.27)) (justify left))
   )
-  (hierarchical_label "DI_3" (shape input) (at 76.2 46.99 90) (fields_autoplaced)
-    (effects (font (size 1.27 1.27)) (justify left))
-  )
-  (hierarchical_label "DI_3_TTL" (shape output) (at 101.6 63.5 90) (fields_autoplaced)
-    (effects (font (size 1.27 1.27)) (justify left))
-  )
-  (hierarchical_label "DI_4" (shape input) (at 53.34 46.99 90) (fields_autoplaced)
-    (effects (font (size 1.27 1.27)) (justify left))
-  )
-  (hierarchical_label "DI_2" (shape input) (at 96.52 46.99 90) (fields_autoplaced)
-    (effects (font (size 1.27 1.27)) (justify left))
-  )
