File: hardware/Radio.kicad_sch (KiCad schematic)
At the start: 39 parts, among them Q801 BC817, U801 RF69, U802 AS193-73LF, Y801 32_Mhz

Commit message: hardware: add USB for debugging and programming
Signed-off-by: Connor Rigby <connorr@hey.com>
Parts:
- U802: footprint Package_TO_SOT_SMD:SOT-363_SC-70-6 -> Package_TO_SOT_SMD:SOT-23-6
Changed lines of the file:
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@@
       (effects (font (size 1.27 1.27)))
     )
-    (property "Footprint" "Package_TO_SOT_SMD:SOT-363_SC-70-6" (at 215.9 107.95 0)
+    (property "Footprint" "Package_TO_SOT_SMD:SOT-23-6" (at 215.9 107.95 0)
       (effects (font (size 1.27 1.27)) hide)
     )

Commit message: Rev 2 submitted for production
Signed-off-by: Connor Rigby <connorr@hey.com>
Parts:
- removed C811, C812: C_0402_33p_C0G, Capacitor_SMD:C_0402_1005Metric, symbol LCSC_Capacitor:C_0402_33p_C0G
- added C811, C812: C_0402_22p_C0G, Capacitor_SMD:C_0402_1005Metric, symbol LCSC_Capacitor:C_0402_22p_C0G
- C801: symbol LCSC_Capacitor:C_0402_10n_C0G -> LCSC_Capacitor:C_0402_10n_X7R; Capacitance 10nf -> 10nF; LCSC C1518210 -> C60133; MPN GRM1555CYA103JE01D -> CC0402KRX7R9BB103; Temperature C0G -> X7R; Tolerance ±5% -> ±10%; Voltage 35V -> 50V
- Y801: LCSC C5143379 -> C9009; MPN TAXM32M4RLBCDT2T -> X322532MOB4SI
Connections:
- net GND: now also C811.1, C812.1
- net XTA: now also C811.2
- net XTB: now also C812.2
- net +3.3V renamed VDD
- net VDD: no longer C813.1, U801.15 (VBAT2)
- new net +BATT: C813.1, U801.15 (VBAT2)
