File: hardware/BLE.kicad_sch (KiCad schematic)
At the start: 33 parts, among them J601 Conn_02x03_Odd_Even, Q801 BC817, U601 ESP32-C3FH4, Y502 Q13FC1350000400, Y601 40_Mhz

Commit message: ughhhhhhhhhhhhhhhhhhhhhhhhhhhhhhhhhhhhhhhhhhhhhhhhhhh
Signed-off-by: Connor Rigby <connorr@hey.com>
Parts:
- removed C603: C_0805_1u_X7R, Capacitor_SMD:C_0805_2012Metric, symbol LCSC_Capacitor:C_0805_1u_X7R
- removed C604: C_0402_10n_C0G, Capacitor_SMD:C_0402_1005Metric, symbol LCSC_Capacitor:C_0402_10n_X7R
- removed C605: C_0805_10u_X5R, Capacitor_SMD:C_0805_2012Metric, symbol LCSC_Capacitor:C_0805_10u_X5R
- removed C610, C612: C_0402_100nf_X7R, Capacitor_SMD:C_0402_1005Metric, symbol LCSC_Capacitor:C_0402_100nf_X7R
- removed C811 (x4): C_0402_22p_C0G, Capacitor_SMD:C_0402_1005Metric, symbol LCSC_Capacitor:C_0402_22p_C0G
- removed J601: Conn_02x03_Odd_Even, Connector:Tag-Connect_TC2030-IDC-NL_2x03_P1.27mm_Vertical, symbol Connector_Generic:Conn_02x03_Odd_Even
- removed L601: L_0402_22n, Inductor_SMD:L_0402_1005Metric, symbol LCSC_Inductor:L_0402_22n
- removed Q801 (x2): BC817, Package_TO_SOT_SMD:SOT-23, symbol LCSC_Transistor1:BC817
- removed R602: R_0603_499, Resistor_SMD:R_0603_1608Metric, symbol LCSC_Resistor:R_0603_499
- removed R603, R604, R605, R608: R_0402_10k, Resistor_SMD:R_0402_1005Metric, symbol LCSC_Resistor:R_0402_10k
- removed U601: ESP32-C3FH4, LCSC_Microcontroller:QFN50P500X500X90-33N, symbol LCSC_Microcontroller:ESP32-C3FH4
- removed Y502: Q13FC1350000400, Crystal:Crystal_SMD_3215-2Pin_3.2x1.5mm, symbol LCSC_Crystal:Q13FC1350000400
- removed Y601: 40_Mhz, Crystal:Crystal_SMD_3225-4Pin_3.2x2.5mm, symbol LCSC_Crystal:40_Mhz
- added C521, C602, C603, C604, C605, C615, C616: C_0402_100nf_X7R, Capacitor_SMD:C_0402_1005Metric, symbol LCSC_Capacitor:C_0402_100nf_X7R
- added C610, C612: C_0805_4u7_X5R, Capacitor_SMD:C_0805_2012Metric, symbol LCSC_Capacitor:C_0805_4u7_X5R
- added FB601: 500mΩ ±25% 600Ω@100MHz 0603 Ferrite Beads, Inductor_SMD:L_0603_1608Metric, symbol Device:FerriteBead_Small
- added L601: 10uH, symbol Device:L_Small
- added L603: 10uH, Inductor_SMD:L_0805_2012Metric, symbol Device:L_Small
- added R502: R_0402_0, Resistor_SMD:R_0402_1005Metric, symbol LCSC_Resistor:R_0402_0
- added R503, R504, R505: R_0402_10k, Resistor_SMD:R_0402_1005Metric, symbol LCSC_Resistor:R_0402_10k
- added U501: W25Q16JVSSIQ, Package_SO:SOIC-8_5.23x5.23mm_P1.27mm, symbol LCSC_Microcontroller:W25Q16JVSSIQ
- added U602: STM32WB15CCU6, Package_DFN_QFN:QFN-48-1EP_7x7mm_P0.5mm_EP5.6x5.6mm, symbol MCU_ST_STM32WB:STM32WB15CCUx
- renumbered AE802 to AE601, C826 to C613, C827 to C614
Connections:
- net GND: now also C521.2, C610.2, C612.2, C615.2, C616.2, U501.4 (GND); no longer C606.2, C607.2
- net VDD: now also C521.1, R503.1, R504.1, R505.1, U501.8 (VCC); no longer C606.1, C611.1
- net VDD3P3: no longer names the net of C607.1
- net VDD3P3: now also FB601.1, U602.8 (VDDA)
- new net: C615.1, C616.1, U602.23 (VDDRF)
- new net: C606.1, U602.1 (VBAT)
- new net: C602.1, C603.1, C604.1, C605.1, U602.20 (VDD), U602.35 (VDD), U602.40 (VDD), U602.48 (VDD)
- new net: L601.2, U602.33 (VLXSMPS)
- new net: L601.1, L603.2
- new net BLE_RESET: U602.7 (NRST(PB11))
- new net FLASH_HOLD: R505.2, U501.7 (IO3)
- new net FLASH_SCK: R502.1, U501.6 (CLK)
- new net FLASH_WP: R504.2, U501.3 (IO2)
- new net HCI.CTS: U602.15 (PA6)
- new net HCI.RTS: U602.29 (PB1)
- new net HCI.RX: U602.12 (PA3)
- new net HCI.TX: U602.11 (PA2)
- new net JT.CK: U602.41 (PA14)
- new net JT.DI: U602.42 (PA15)
- new net JT.DO: U602.43 (PB3)
- new net JT.MS: U602.39 (PA13)
- new net JT.RST: U602.44 (PB4)
- new net RCC_OSC32_IN: U602.2 (PC14)
- new net RCC_OSC32_OUT: U602.3 (PC15)
- new net RCC_OSC_IN: U602.24 (OSC_OUT)
- new net RCC_OSC_OUT: U602.25 (OSC_IN)
- new net SPI1.MISO: U501.2 (DO(IO1))
- new net SPI1.MOSI: U501.5 (DI(IO0))
- new net SPI1.NSS: R503.2, U501.1 (~{CS})
- new net SPI1.SCK: R502.2
- new net VCP.RX: U602.47 (PB7)
- new net VCP.TX: U602.5 (PB8)
- new net VDDSMPS: C610.1, C611.1, C612.1, L603.1, U602.31 (VFBSMPS), U602.34 (VDDSMPS)
- no-connect marks 14 -> 2
Other:
- note added: "https://www.lcsc.com/product-detail/RF-Filters_STMicroelectronics-MLPF-WB-01E3_C3155642.html"

Commit message: asdf
Signed-off-by: Connor Rigby <connorr@hey.com>
Parts:
- removed C613, C614: C_0402_DNP, Capacitor_SMD:C_0402_1005Metric, symbol LCSC_Capacitor:C_0402_DNP
- removed R601: R_0402_0, Resistor_SMD:R_0402_1005Metric, symbol LCSC_Resistor:R_0402_0
- added C507, C508, C509, C510: C_0402_DNP, Capacitor_SMD:C_0402_1005Metric, symbol LCSC_Capacitor:C_0402_DNP
- added U603: MLPF-WB-01E3, LCSC_Antenna:CSP6_BUMPLESS_STM, symbol LCSC_Antenna:MLPF-WB-01E3
- added Y501: 32_Mhz, Crystal:Crystal_SMD_3225-4Pin_3.2x2.5mm, symbol LCSC_Crystal:32_Mhz
- added Y502: Q13FC1350000400, footprint:FC-135R_L3.2-W1.5, symbol LCSC_Crystal:Q13FC1350000400
Connections:
- net BLE_ANT is gone; now on net BT_ANT: ANT601.1 (SIG)
- net GND: now also C602.2, C603.2, C604.2, C605.2, C606.2, C607.2, U602.22 (VSSRF), U602.32 (VSSSMPS), U602.49 (VSS), C507.2, C508.2, C509.2, C510.2, U603.A1 (OUT), U603.B1 (GND4), U603.B2 (GND2), U603.C2 (GND1), Y501.2, Y501.4
- net LNA_IN: now also U603.A2 (GND3)
- net RCC_OSC32_IN: now also C509.1, Y502.1
- net RCC_OSC32_OUT: now also C510.1, Y502.2
- net RCC_OSC_IN: now also C507.1, Y501.1
- net RCC_OSC_OUT: now also C508.1, Y501.3
- net VDD: now also C602.1, C603.1, C604.1, C605.1, C615.1, C616.1, FB601.2, U602.20 (VDD), U602.23 (VDDRF), U602.35 (VDD), U602.40 (VDD), U602.48 (VDD)
- net +BATT: now reaches C606.1, U602.1 (VBAT)
- net at U602.21 (RF1): now also U603.C1 (IN)
- net VDDA: now reaches C607.1, FB601.1, U602.8 (VDDA)
- net BLE_RESET renamed ~{RESET}
Other:
- note removed: "https://www.lcsc.com/product-detail/RF-Filters_STMicroelectronics-MLPF-WB-01E3_C3155642.html"
- moved on the sheet: AE601, AE602, C612

Commit message: updates
Signed-off-by: Connor Rigby <connorr@hey.com>
Parts:
- L601: footprint (none) -> Inductor_SMD:L_0805_2012Metric_Pad1.15x1.40mm_HandSolder; MPN (none) -> 74479777310A
- L603: footprint Inductor_SMD:L_0805_2012Metric -> Inductor_SMD:L_0805_2012Metric_Pad1.15x1.40mm_HandSolder
- Y502: footprint footprint:FC-135R_L3.2-W1.5 -> Crystal:Crystal_SMD_3215-2Pin_3.2x1.5mm
Connections:
- net SPI1.MISO: now also U602.37 (PA11)
- net SPI1.MOSI: now also U602.14 (PA5)
- net SPI1.NSS: now also U602.13 (PA4)
- net SPI1.SCK: now also U602.10 (PA1)
- net VDDA: no longer names the net of C607.1, FB601.1, U602.8 (VDDA)
- no-connect marks 2 -> 15
Changed lines of the file:
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@@
   (junction (at 198.12 31.75) (diameter 0) (color 0 0 0 0)
   )
+  (junction (at 224.79 40.64) (diameter 0) (color 0 0 0 0)
+  )
   (junction (at 193.04 31.75) (diameter 0) (color 0 0 0 0)
   )
@@
   (junction (at 279.4 49.53) (diameter 0) (color 0 0 0 0)
   )
-  (junction (at 200.66 40.64) (diameter 0) (color 0 0 0 0)
-  )
   (junction (at 50.8 114.3) (diameter 0) (color 0 0 0 0)
   )
@@
   (junction (at 50.8 50.8) (diameter 0) (color 0 0 0 0)
   )
+  (no_connect (at 218.44 83.82))
+  (no_connect (at 218.44 76.2))
+  (no_connect (at 218.44 88.9))
+  (no_connect (at 218.44 58.42))
+  (no_connect (at 218.44 124.46))
+  (no_connect (at 218.44 116.84))
+  (no_connect (at 172.72 91.44))
+  (no_connect (at 172.72 86.36))
+  (no_connect (at 218.44 101.6))
   (no_connect (at 114.3 44.45))
+  (no_connect (at 218.44 106.68))
+  (no_connect (at 218.44 78.74))
   (no_connect (at 139.7 44.45))
+  (no_connect (at 218.44 81.28))
+  (no_connect (at 218.44 114.3))
   (wire (pts (xy 139.7 76.2) (xy 139.7 72.39))
     (stroke (width 0) (type default))
@@
     (stroke (width 0) (type default))
   )
+  (wire (pts (xy 218.44 71.12) (xy 232.41 71.12))
+    (stroke (width 0) (type default))
+  )
+  (wire (pts (xy 218.44 68.58) (xy 232.41 68.58))
+    (stroke (width 0) (type default))
+  )
   (wire (pts (xy 115.57 114.3) (xy 114.3 114.3))
     (stroke (width 0) (type default))
@@
     (stroke (width 0) (type default))
   )
+  (wire (pts (xy 218.44 86.36) (xy 232.41 86.36))
+    (stroke (width 0) (type default))
+  )
   (wire (pts (xy 76.2 157.48) (xy 101.6 157.48))
     (stroke (width 0) (type default))
@@
   )
   (wire (pts (xy 187.96 53.34) (xy 187.96 31.75))
+    (stroke (width 0) (type default))
+  )
+  (wire (pts (xy 218.44 60.96) (xy 232.41 60.96))
     (stroke (width 0) (type default))
   )
@@
     )
   )
+  (label "SPI1.MISO" (at 232.41 86.36 180) (fields_autoplaced)
+    (effects (font (size 1.27 1.27)) (justify right bottom))
+    (property "Netclass" "SPI" (at 232.41 87.63 0)
+      (effects (font (size 1.27 1.27) italic) (justify right) hide)
+    )
+  )
   (label "LNA_IN" (at 63.5 50.8 180) (fields_autoplaced)
     (effects (font (size 1.27 1.27)) (justify right bottom))
+  )
+  (label "SPI1.SCK" (at 232.41 60.96 180) (fields_autoplaced)
+    (effects (font (size 1.27 1.27)) (justify right bottom))
+    (property "Netclass" "SPI" (at 232.41 62.23 0)
+      (effects (font (size 1.27 1.27) italic) (justify right) hide)
+    )
   )
   (label "SPI1.NSS" (at 50.8 162.56 0) (fields_autoplaced)
@@
   (label "RCC_OSC_IN" (at 152.4 71.12 0) (fields_autoplaced)
     (effects (font (size 1.27 1.27)) (justify left bottom))
-    (property "Netclass" "GPIO" (at 152.4 72.39 0)
+    (property "Netclass" "RCC" (at 152.4 72.39 0)
       (effects (font (size 1.27 1.27) italic) (justify left) hide)
     )
@@
     )
   )
+  (label "SPI1.NSS" (at 232.41 68.58 180) (fields_autoplaced)
+    (effects (font (size 1.27 1.27)) (justify right bottom))
+    (property "Netclass" "SPI" (at 232.41 69.85 0)
+      (effects (font (size 1.27 1.27) italic) (justify right) hide)
+    )
+  )
   (label "RCC_OSC_OUT" (at 152.4 68.58 0) (fields_autoplaced)
     (effects (font (size 1.27 1.27)) (justify left bottom))
-    (property "Netclass" "GPIO" (at 152.4 69.85 0)
+    (property "Netclass" "RCC" (at 152.4 69.85 0)
       (effects (font (size 1.27 1.27) italic) (justify left) hide)
     )
@@
   (label "BT_ANT" (at 25.4 50.8 0) (fields_autoplaced)
     (effects (font (size 1.27 1.27)) (justify left bottom))
+  )
+  (label "SPI1.MOSI" (at 232.41 71.12 180) (fields_autoplaced)
+    (effects (font (size 1.27 1.27)) (justify right bottom))
+    (property "Netclass" "SPI" (at 232.41 72.39 0)
+      (effects (font (size 1.27 1.27) italic) (justify right) hide)
+    )
   )
   (label "VDDSMPS" (at 205.74 50.8 0) (fields_autoplaced)
@@
       (effects (font (size 1.27 1.27)))
     )
-    (property "Footprint" "" (at 146.05 63.5 0)
+    (property "Footprint" "Inductor_SMD:L_0805_2012Metric_Pad1.15x1.40mm_HandSolder" (at 146.05 63.5 0)
       (effects (font (size 1.27 1.27)) hide)
     )
     (property "Datasheet" "~" (at 146.05 63.5 0)
+      (effects (font (size 1.27 1.27)) hide)
+    )
+    (property "MPN" "74479777310A" (at 146.05 63.5 90)
       (effects (font (size 1.27 1.27)) hide)
     )
@@
       (effects (font (size 1.27 1.27)) hide)
     )
-    (property "Footprint" "footprint:FC-135R_L3.2-W1.5" (at 118.11 114.3 0)
+    (property "Footprint" "Crystal:Crystal_SMD_3215-2Pin_3.2x1.5mm" (at 118.11 114.3 0)
       (effects (font (size 1.27 1.27) italic) hide)
     )
@@
       (effects (font (size 1.27 1.27)) (justify right))
     )
-    (property "Footprint" "Inductor_SMD:L_0805_2012Metric" (at 139.7 69.85 0)
+    (property "Footprint" "Inductor_SMD:L_0805_2012Metric_Pad1.15x1.40mm_HandSolder" (at 139.7 69.85 0)
       (effects (font (size 1.27 1.27)) hide)
     )
@@
     )
   )
+  (symbol (lib_id "power:PWR_FLAG") (at 224.79 40.64 0) (unit 1)
+    (in_bom yes) (on_board yes) (dnp no)
+    (property "Reference" "#FLG0601" (at 224.79 38.735 0)
+      (effects (font (size 1.27 1.27)) hide)
+    )
+    (property "Value" "PWR_FLAG" (at 219.71 39.37 0)
+      (effects (font (size 1.27 1.27)))
+    )
+    (property "Footprint" "" (at 224.79 40.64 0)
+      (effects (font (size 1.27 1.27)) hide)
+    )
+    (property "Datasheet" "~" (at 224.79 40.64 0)
+      (effects (font (size 1.27 1.27)) hide)
+    )
+    (pin "1")
+    (instances
+      (project "underglow2"
+        (path "/dcbdf88a-d6ac-4b1d-9514-0b0ce113d90b/f6dd0682-1649-403c-b931-941640049f3a"
+          (reference "#FLG0601") (unit 1)
+        )
+      )
+    )
+  )
   (symbol (lib_id "LCSC_Capacitor:C_0402_1p8_C0G") (at 25.4 53.34 0) (mirror y) (unit 1)
     (in_bom yes) (on_board yes) (dnp no) (fields_autoplaced)
@@
         )
       )
-    )
-  )
-  (symbol (lib_id "power:VDDA") (at 200.66 40.64 0) (unit 1)
-    (in_bom yes) (on_board yes) (dnp no) (fields_autoplaced)
-    (property "Reference" "#PWR0629" (at 200.66 44.45 0)
-      (effects (font (size 1.27 1.27)) hide)
-    )
-    (property "Value" "VDDA" (at 200.66 36.83 0)
-      (effects (font (size 1.27 1.27)))
-    )
-    (property "Footprint" "" (at 200.66 40.64 0)
-      (effects (font (size 1.27 1.27)) hide)
-    )
-    (property "Datasheet" "" (at 200.66 40.64 0)
-      (effects (font (size 1.27 1.27)) hide)
-    )
-    (pin "1")
-    (instances
-      (project "underglow2"
-        (path "/dcbdf88a-d6ac-4b1d-9514-0b0ce113d90b/f6dd0682-1649-403c-b931-941640049f3a"
-          (reference "#PWR0629") (unit 1)
-        )
-      )
