File: hardware/Debugger.kicad_sch (KiCad schematic)
At the start: 5 parts, among them J501 Conn_ST_STDC14

Commit message: asdf
Signed-off-by: Connor Rigby <connorr@hey.com>
Parts:
- removed JP501: SolderJumper_3_Open, Jumper:SolderJumper-3_P1.3mm_Open_RoundedPad1.0x1.5mm_NumberLabels, symbol Jumper:SolderJumper_3_Open
- added SW801: VCP, symbol Switch:SW_DIP_x04
- added SW802: SW_DIP_x02, symbol Switch:SW_DIP_x02
Connections:
- net SYS_JTDI is gone; now on net JT.DI: J501.10 (JTDI/NC)
- net SYS_JTDO is gone; now on net JT.DO: J501.8 (JTDO/SWO)
- net SYS_JTMS is gone; now on net JT.MS: J501.4 (JTMS/SWDIO)
- net JT.RST: now also SW802.1
- net ~{DEBUG_RST}: now also SW802.3, SW802.4
- net SYS_JTCK renamed JT.CK
- net USART1_RX renamed VCP.RX
- net VCP.RX: now also SW801.7, SW801.8
- net USART1_TX renamed VCP.TX
- net VCP.TX: now also SW801.5, SW801.6
- net ~{RST} renamed ~{RESET}
- net ~{RESET}: now also SW802.2
- new net VCP1.RX: SW801.1
- new net VCP1.TX: SW801.2
- new net VCP2.RX: SW801.3
- new net VCP2.TX: SW801.4
Other:
- company: (none) -> https://cone.codes
- title: (none) -> coneRGB2
- moved on the sheet: C516, C520, D202, J501

Commit message: updates
Signed-off-by: Connor Rigby <connorr@hey.com>
Parts:
- SW801: footprint (none) -> Button:SW-SMD_8P-L6.7-W5.4-P1.27-LS8.4
- SW802: footprint (none) -> Button:SW-SMD_4P_DSHP02TSGET; LCSC (none) -> C40735
Changed lines of the file:
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@@
       (effects (font (size 1.27 1.27)))
     )
-    (property "Footprint" "" (at 55.88 44.45 0)
+    (property "Footprint" "Button:SW-SMD_4P_DSHP02TSGET" (at 55.88 44.45 0)
       (effects (font (size 1.27 1.27)) hide)
     )
     (property "Datasheet" "~" (at 55.88 44.45 0)
+      (effects (font (size 1.27 1.27)) hide)
+    )
+    (property "LCSC" "C40735" (at 55.88 44.45 0)
       (effects (font (size 1.27 1.27)) hide)
     )
@@
       (effects (font (size 1.27 1.27)))
     )
-    (property "Footprint" "" (at 55.88 71.12 0)
+    (property "Footprint" "Button:SW-SMD_8P-L6.7-W5.4-P1.27-LS8.4" (at 55.88 71.12 0)
       (effects (font (size 1.27 1.27)) hide)
     )
