File: hardware/Power.kicad_sch (KiCad schematic)
At the start: 14 parts, among them U201 AMS1117-5.0, U202 AMS1117-3.3

Commit message: updates
Signed-off-by: Connor Rigby <connorr@hey.com>
Changed lines of the file:
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@@
   (junction (at 50.8 38.1) (diameter 0) (color 0 0 0 0)
+  )
+  (junction (at 50.8 25.4) (diameter 0) (color 0 0 0 0)
   )
   (junction (at 119.38 38.1) (diameter 0) (color 0 0 0 0)
@@
         )
       )
+    )
+  )
+  (symbol (lib_id "power:PWR_FLAG") (at 50.8 25.4 0) (unit 1)
+    (in_bom yes) (on_board yes) (dnp no) (fields_autoplaced)
+    (property "Reference" "#FLG0201" (at 50.8 23.495 0)
+      (effects (font (size 1.27 1.27)) hide)
+    )
+    (property "Value" "PWR_FLAG" (at 50.8 20.32 0)
+      (effects (font (size 1.27 1.27)))
+    )
+    (property "Footprint" "" (at 50.8 25.4 0)
+      (effects (font (size 1.27 1.27)) hide)
+    )
+    (property "Datasheet" "~" (at 50.8 25.4 0)
+      (effects (font (size 1.27 1.27)) hide)
+    )
+    (pin "1")
+    (instances
+      (project "underglow2"
+        (path "/dcbdf88a-d6ac-4b1d-9514-0b0ce113d90b/51e4e0b8-920f-4548-a9c8-d97d830c9625"
+          (reference "#FLG0201") (unit 1)
+        )
+      )
