File: hardware/RGB.kicad_sch (KiCad schematic)
At the start: 16 parts, among them Q301 Q_PMOS_GDS, Q302 Q_NMOS_GDS, Q303 Q_NMOS_GDS, Q304 Q_NMOS_GDS, U301 MCP1416, U302 MCP1416, U303 MCP1416

Commit message: updates
Signed-off-by: Connor Rigby <connorr@hey.com>
Parts:
- added R305, R306, R307: R_0603_DNP, Resistor_SMD:R_0603_1608Metric, symbol LCSC_Resistor:R_0603_DNP
Connections:
- net B_PWM_IN: now also R307.1; no longer R304.1, U303.3 (IN)
- net G_PWM_IN: now also R306.1; no longer R303.1, U302.3 (IN)
- net R_PWM_IN: now also R305.1; no longer R302.1, U301.3 (IN)
- new net: R302.1, R305.2, U301.3 (IN)
- new net: R304.1, R307.2, U303.3 (IN)
- new net: R303.1, R306.2, U302.3 (IN)
Changed lines of the file:
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@@
   (junction (at 215.9 76.2) (diameter 0) (color 0 0 0 0)
   )
+  (junction (at 224.79 101.6) (diameter 0) (color 0 0 0 0)
+  )
   (junction (at 236.22 76.2) (diameter 0) (color 0 0 0 0)
   )
   (junction (at 127 76.2) (diameter 0) (color 0 0 0 0)
   )
+  (junction (at 34.29 101.6) (diameter 0) (color 0 0 0 0)
+  )
+  (junction (at 45.72 57.15) (diameter 0) (color 0 0 0 0)
+  )
+  (junction (at 135.89 101.6) (diameter 0) (color 0 0 0 0)
+  )
   (wire (pts (xy 215.9 76.2) (xy 236.22 76.2))
     (stroke (width 0) (type default))
@@
     (stroke (width 0) (type default))
   )
-  (wire (pts (xy 45.72 55.88) (xy 45.72 76.2))
+  (wire (pts (xy 45.72 55.88) (xy 45.72 57.15))
     (stroke (width 0) (type default))
   )
@@
   )
   (wire (pts (xy 25.4 76.2) (xy 45.72 76.2))
+    (stroke (width 0) (type default))
+  )
+  (wire (pts (xy 45.72 57.15) (xy 45.72 76.2))
     (stroke (width 0) (type default))
   )
@@
     )
   )
-  (hierarchical_label "R_PWM_IN" (shape input) (at 34.29 101.6 180) (fields_autoplaced)
+  (hierarchical_label "R_PWM_IN" (shape input) (at 29.21 101.6 180) (fields_autoplaced)
     (effects (font (size 1.27 1.27)) (justify right))
-    (property "Netclass" "PWM" (at 34.29 102.87 0)
+    (property "Netclass" "PWM" (at 29.21 102.87 0)
       (effects (font (size 1.27 1.27) italic) (justify right) hide)
     )
   )
-  (hierarchical_label "G_PWM_IN" (shape input) (at 135.89 101.6 180) (fields_autoplaced)
+  (hierarchical_label "G_PWM_IN" (shape input) (at 130.81 101.6 180) (fields_autoplaced)
     (effects (font (size 1.27 1.27)) (justify right))
-    (property "Netclass" "PWM" (at 135.89 102.87 0)
+    (property "Netclass" "PWM" (at 130.81 102.87 0)
       (effects (font (size 1.27 1.27) italic) (justify right) hide)
     )
   )
-  (hierarchical_label "B_PWM_IN" (shape input) (at 224.79 101.6 180) (fields_autoplaced)
+  (hierarchical_label "B_PWM_IN" (shape input) (at 219.71 101.6 180) (fields_autoplaced)
     (effects (font (size 1.27 1.27)) (justify right))
-    (property "Netclass" "PWM" (at 224.79 102.87 0)
+    (property "Netclass" "PWM" (at 219.71 102.87 0)
       (effects (font (size 1.27 1.27) italic) (justify right) hide)
     )
@@
     )
   )
+  (symbol (lib_id "LCSC_Resistor:R_0603_DNP") (at 31.75 101.6 90) (unit 1)
+    (in_bom no) (on_board yes) (dnp no) (fields_autoplaced)
+    (property "Reference" "R305" (at 31.75 96.52 90)
+      (effects (font (size 1.27 1.27)))
+    )
+    (property "Value" "R_0603_DNP" (at 31.75 99.06 90)
+      (effects (font (size 1.27 1.27)))
+    )
+    (property "Footprint" "Resistor_SMD:R_0603_1608Metric" (at 31.75 101.6 0)
+      (effects (font (size 1.27 1.27)) hide)
+    )
+    (property "Datasheet" "~" (at 31.75 101.6 0)
+      (effects (font (size 1.27 1.27)) hide)
+    )
+    (pin "1")
+    (pin "2")
+    (instances
+      (project "underglow2"
+        (path "/dcbdf88a-d6ac-4b1d-9514-0b0ce113d90b/d698d388-4189-4a55-a8ce-744fe305194e"
+          (reference "R305") (unit 1)
+        )
+      )
+    )
+  )
   (symbol (lib_id "power:GND") (at 215.9 81.28 0) (unit 1)
     (in_bom yes) (on_board yes) (dnp no) (fields_autoplaced)
@@
     )
   )
+  (symbol (lib_id "LCSC_Resistor:R_0603_DNP") (at 222.25 101.6 90) (unit 1)
+    (in_bom no) (on_board yes) (dnp no) (fields_autoplaced)
+    (property "Reference" "R307" (at 222.25 96.52 90)
+      (effects (font (size 1.27 1.27)))
+    )
+    (property "Value" "R_0603_DNP" (at 222.25 99.06 90)
+      (effects (font (size 1.27 1.27)))
+    )
+    (property "Footprint" "Resistor_SMD:R_0603_1608Metric" (at 222.25 101.6 0)
+      (effects (font (size 1.27 1.27)) hide)
+    )
+    (property "Datasheet" "~" (at 222.25 101.6 0)
+      (effects (font (size 1.27 1.27)) hide)
+    )
+    (pin "1")
+    (pin "2")
+    (instances
+      (project "underglow2"
+        (path "/dcbdf88a-d6ac-4b1d-9514-0b0ce113d90b/d698d388-4189-4a55-a8ce-744fe305194e"
+          (reference "R307") (unit 1)
+        )
+      )
+    )
+  )
   (symbol (lib_id "LCSC_Resistor:R_0603_100k") (at 135.89 107.95 0) (unit 1)
     (in_bom yes) (on_board yes) (dnp no)
@@
     )
   )
+  (symbol (lib_id "LCSC_Resistor:R_0603_DNP") (at 133.35 101.6 90) (unit 1)
+    (in_bom no) (on_board yes) (dnp no) (fields_autoplaced)
+    (property "Reference" "R306" (at 133.35 96.52 90)
+      (effects (font (size 1.27 1.27)))
+    )
+    (property "Value" "R_0603_DNP" (at 133.35 99.06 90)
+      (effects (font (size 1.27 1.27)))
+    )
+    (property "Footprint" "Resistor_SMD:R_0603_1608Metric" (at 133.35 101.6 0)
+      (effects (font (size 1.27 1.27)) hide)
+    )
+    (property "Datasheet" "~" (at 133.35 101.6 0)
+      (effects (font (size 1.27 1.27)) hide)
+    )
+    (pin "1")
+    (pin "2")
+    (instances
+      (project "underglow2"
+        (path "/dcbdf88a-d6ac-4b1d-9514-0b0ce113d90b/d698d388-4189-4a55-a8ce-744fe305194e"
+          (reference "R306") (unit 1)
+        )
+      )
+    )
+  )
   (symbol (lib_id "power:+12V") (at 45.72 45.72 0) (unit 1)
     (in_bom yes) (on_board yes) (dnp no) (fields_autoplaced)
@@
         )
       )
+    )
+  )
+  (symbol (lib_id "power:PWR_FLAG") (at 45.72 57.15 90) (unit 1)
+    (in_bom yes) (on_board yes) (dnp no) (fields_autoplaced)
+    (property "Reference" "#FLG0301" (at 43.815 57.15 0)
+      (effects (font (size 1.27 1.27)) hide)
+    )
+    (property "Value" "PWR_FLAG" (at 41.91 57.15 90)
+      (effects (font (size 1.27 1.27)) (justify left))
+    )
+    (property "Footprint" "" (at 45.72 57.15 0)
+      (effects (font (size 1.27 1.27)) hide)
+    )
+    (property "Datasheet" "~" (at 45.72 57.15 0)
+      (effects (font (size 1.27 1.27)) hide)
+    )
+    (pin "1")
+    (instances
+      (project "underglow2"
+        (path "/dcbdf88a-d6ac-4b1d-9514-0b0ce113d90b/d698d388-4189-4a55-a8ce-744fe305194e"
+          (reference "#FLG0301") (unit 1)
+        )
+      )
