File: hardware/underglow2.kicad_sch (KiCad schematic)
At the start: 1 part, among them J101 J_Delphi_Sicma_24

Commit message: ughhhhhhhhhhhhhhhhhhhhhhhhhhhhhhhhhhhhhhhhhhhhhhhhhhh
Signed-off-by: Connor Rigby <connorr@hey.com>
Connections:
- net CAN/CAN_H: no longer J101.B3
- net CAN/CAN_L: no longer J101.B4
- net Digital Input/DI_1: no longer J101.C2
- net Digital Input/DI_2: no longer J101.C3
- net Digital Input/DI_3: no longer J101.C4
- net Digital Input/DI_4: no longer J101.C5
- net RGB/PIXEL_1: no longer J101.C6
- net RGB/PIXEL_2: no longer J101.C7
- net RGB/RGB1_12V: no longer J101.C1
- net RGB/RGB1_B: no longer J101.A4
- net RGB/RGB1_G: no longer J101.A3
- net RGB/RGB1_R: no longer J101.A2
- net RGB/RGB2_12V: no longer J101.B1
- net RGB/RGB2_B: no longer J101.A7
- net RGB/RGB2_G: no longer J101.A6
- net RGB/RGB2_R: no longer J101.A5
- net Power/EN: no longer names the net of J101.B2
Other:
- removed sheet Radio
- added sheet Debugger (Debugger.kicad_sch)
- sheet Application ports: added JT.DI, JT.DO, JT.MS, JT.RST, JT.TCK; removed RADIO_IRQ, RADIO_MISO, RADIO_MOSI, RADIO_NSS, RADIO_SCK, ~{RADIO_RESET}
- sheet BLE ports: added JT.DI, JT.DO, JT.MS, JT.RST, JT.TCK; removed none
- sheet Power ports: added none; removed EN
- moved on the sheet: J101

Commit message: asdf
Signed-off-by: Connor Rigby <connorr@hey.com>
Connections:
- net R_PWM_OUT: now reaches J101.A2
- net R_PWM_OUT: now also J101.A5
- net G_PWM_OUT: now reaches J101.A3
- net G_PWM_OUT: now also J101.A6
- net B_PWM_OUT: now reaches J101.A4
- net B_PWM_OUT: now also J101.A7
- net RGB_VOUT: now reaches J101.B1
- net RGB_VOUT: now also J101.C1
- net RGB_EN: now reaches J101.B2
- net CAN_H: now reaches J101.B3
- net CAN_L: now reaches J101.B4
- net PI4: now reaches J101.C2
- net PI3: now reaches J101.C3
- net PI2: now reaches J101.C4
- net PI1: now reaches J101.C5
- net NZR2_OUT: now reaches J101.C6
- net NZR1_OUT: now reaches J101.C7
Other:
- sheet Application ports: added B_PWM, G_PWM, HCI.CTS, HCI.RTS, HCI.RX, HCI.TX, JT.CK, NZR1_PWM, NZR2_PWM, R_PWM, VCP_RX, VCP_TX, ~{RESET}; removed CH1_B_PWM, CH1_EN_PWM, CH1_G_PWM, CH1_NZR, CH1_R_PWM, CH2_B_PWM, CH2_EN_PWM, CH2_G_PWM, CH2_NZR, CH2_R_PWM, HCI_CTS, HCI_EN, HCI_RTS, HCI_RX, HCI_TX, JT.TCK
- sheet BLE ports: added HCI.CTS, HCI.RTS, HCI.RX, HCI.TX, JT.CK, VCP.RX, VCP.TX, ~{RESET}; removed HCI_CTS, HCI_EN, HCI_RTS, HCI_RX, HCI_TX, JT.TCK
- sheet Debugger ports: added VCP1.RX, VCP1.TX, VCP2.RX, VCP2.TX, ~{RESET}; removed none
- sheet RGB ports: added B_PWM_IN, B_PWM_OUT, G_PWM_IN, G_PWM_OUT, NZR1_IN, NZR1_OUT, NZR2_IN, NZR2_OUT, RGB_EN, RGB_VOUT, R_PWM_IN, R_PWM_OUT; removed CH1_B_PWM, CH1_EN_PWM, CH1_G_PWM, CH1_NZR, CH1_R_PWM, CH2_B_PWM, CH2_EN_PWM, CH2_G_PWM, CH2_NZR, CH2_R_PWM, PIXEL_1, PIXEL_2, RGB1_12V, RGB1_B, RGB1_G, RGB1_R, RGB2_12V, RGB2_B, RGB2_G, RGB2_R
- moved on the sheet: J101

Commit message: updates
Signed-off-by: Connor Rigby <connorr@hey.com>
Changed lines of the file:
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@@
     )
   )
-  (sheet (at 165.1 38.1) (size 25.4 26.67) (fields_autoplaced)
+  (sheet (at 165.1 31.75) (size 25.4 26.67) (fields_autoplaced)
     (stroke (width 0.1524) (type solid))
     (fill (color 0 0 0 0.0000))
-    (property "Sheetname" "Power" (at 165.1 37.3884 0)
+    (property "Sheetname" "Power" (at 165.1 31.0384 0)
       (effects (font (size 1.27 1.27)) (justify left bottom))
     )
-    (property "Sheetfile" "Power.kicad_sch" (at 165.1 65.3546 0)
+    (property "Sheetfile" "Power.kicad_sch" (at 165.1 59.0046 0)
       (effects (font (size 1.27 1.27)) (justify left top) hide)
     )

Commit message: updates
Signed-off-by: Connor Rigby <connorr@hey.com>
Parts:
- removed J101: J_Delphi_Sicma_24, bom:Delphi_Sicma_24_Black, symbol bom:J_Delphi_Sicma_24
- added AE101: Antenna_Chip, LCSC_Antenna:ANT-SMD_L3.2-W1.6, symbol Device:Antenna_Chip
- added C101, C106, C113, C116, C117: C_0805_1u_X7R, Capacitor_SMD:C_0805_2012Metric, symbol LCSC_Capacitor:C_0805_1u_X7R
- added C102, C103, C109, C114, C115, C120, C123 (x2): C_0402_100nf_X7R, Capacitor_SMD:C_0402_1005Metric, symbol LCSC_Capacitor:C_0402_100nf_X7R
- added C104, C105, C110, C111, C112: C_0402_DNP, Capacitor_SMD:C_0402_1005Metric, symbol LCSC_Capacitor:C_0402_DNP
- added C107: C_0402_10n_C0G, Capacitor_SMD:C_0402_1005Metric, symbol LCSC_Capacitor:C_0402_10n_C0G
- added C108: C_0805_10u_X5R, Capacitor_SMD:C_0805_2012Metric, symbol LCSC_Capacitor:C_0805_10u_X5R
- added D101, D104, D105, D106: LED_0603_RED, LED_SMD:LED_0603_1608Metric, symbol LCSC_LED:LED_0603_RED
- added D102, D107, D108, D109, D110, D111, D112: 1N5819WS, Diode_SMD:D_SOD-323, symbol Diode:1N5819WS
- added FB101: FerriteBead_Small, Inductor_SMD:L_0805_2012Metric, symbol Device:FerriteBead_Small
- added H101, H102, H103: SMTSO2020CTJ, LCSC_Connector:SMTSO2020CTJ, symbol Mechanical:MountingHole_Pad
- added J101: Conn_ST_STDC14, LCSC_Connector:TC2070-IDC-FP, symbol Connector:Conn_ST_STDC14
- added J102: ZE05H-16DP-2H, LCSC_Connector:ZE05H-16DP-2H, symbol Connector_Generic_MountingPin:Conn_01x16_MountingPin
- added J103: ZE05-16DS-HU/R, LCSC_Connector:ZE05H-16DP-2H, symbol Connector_Generic_MountingPin:Conn_01x16_MountingPin
- added L101, L102: L_Small, Inductor_SMD:L_0402_1005Metric, symbol Device:L_Small
- added Q101: AO3401A, Package_TO_SOT_SMD:SOT-23, symbol Transistor_FET:AO3401A
- added Q102, Q103, Q104: AO3400A, Package_TO_SOT_SMD:SOT-23, symbol Transistor_FET:AO3400A
- added R101, R108, R109, R110: 100, Resistor_SMD:R_0805_2012Metric, symbol LCSC_Resistor:R_0805_DNP
- added R102, R113, R115, R116: R_0805_10k, Resistor_SMD:R_0805_2012Metric, symbol LCSC_Resistor:R_0805_10k
- added R103, R114, R117, R118: 1k, Resistor_SMD:R_0603_1608Metric, symbol LCSC_Resistor:R_0603_DNP
- added R104, R105, R106, R107: 100, Resistor_SMD:R_0603_1608Metric, symbol LCSC_Resistor:R_0603_DNP
- added R111: 220, Resistor_SMD:R_0805_2012Metric, symbol LCSC_Resistor:R_0805_DNP
- added R119, R123, R124, R125: R_0402_1k, Resistor_SMD:R_0402_1005Metric, symbol LCSC_Resistor:R_0402_1k
- added R120: R_1206_DNP, Resistor_SMD:R_1206_3216Metric, symbol LCSC_Resistor:R_1206_DNP
- added R121: R_0402_DNP, Resistor_SMD:R_0402_1005Metric, symbol LCSC_Resistor:R_0402_DNP
- added R122: R_0402_499, Resistor_SMD:R_0402_1005Metric, symbol LCSC_Resistor:R_0402_499
- added T101, T102, T103, T104, T105, T106, T107, T108, T109, T110, T111, T112, T113, T114, T115, T116: ZE05-2022SCF, symbol Connector:Conn_01x01_Pin
- added U101: ESP32-C3FH4, LCSC_Microcontroller:QFN50P500X500X90-33N, symbol LCSC_Microcontroller:ESP32-C3FH4
- added U102: SN65HVD230, Package_SO:SOIC-8_3.9x4.9mm_P1.27mm, symbol Interface_CAN_LIN:SN65HVD230
- added U103: AMS1117-3.3, Package_TO_SOT_SMD:SOT-223-3_TabPin2, symbol Regulator_Linear:AMS1117-3.3
- added Y101: 40_Mhz, Crystal:Crystal_SMD_3225-4Pin_3.2x2.5mm, symbol LCSC_Crystal:40_Mhz
Connections:
- net CAN_H: now also J102.14 (Pin_14), R120.1, U102.7 (CANH)
- net CAN_L: now also J102.13 (Pin_13), R120.2, U102.6 (CANL)
- net GND: now also AE101.1 (FEED), C101.2, C102.2, C103.2, C104.2, C105.2, C106.2, C107.2, C108.2, C109.2, C110.2, C111.2, C112.2, C113.2, C114.2, C115.2, C116.2, C117.2, C120.2, C123.2, C123.2, D101.1 (K), D104.1 (K), D105.1 (K), D106.1 (K), J101.11 (GNDDetect), J101.5 (GND), J101.7 (GND), J102.12 (Pin_12), J102.3 (Pin_3), J102.4 (Pin_4), Q102.2 (S), Q103.2 (S), Q104.2 (S), R119.2, U101.33 (GND), U102.2 (GND), U103.1 (GND), Y101.2, Y101.4
- net NZR1_OUT: now also D102.1 (K), J102.10 (Pin_10), J102.9 (Pin_9)
- net PI1: now also J102.8 (Pin_8), R102.1
- net PI2: now also J102.2 (Pin_2), R113.1
- net PI3: now also J102.7 (Pin_7), R115.1
- net PI4: now also J102.1 (Pin_1), R116.1
- new net: R119.1, U102.8 (Rs)
- new net: C123.1, D109.1 (K), J101.3 (VCC)
- new net: D102.2 (A), R111.2
- new net: Q101.1 (G), R104.2
- new net: Q101.2 (S), R101.1
- new net: R125.2, U101.14 (GPIO8)
- new net: C110.1, L101.1, U101.2 (VDD3P3), U101.3 (VDD3P3)
- new net: R124.2, U101.6 (GPIO2)
- new net: R102.2, R103.1
- new net: Q102.3 (D), R108.1
- new net: Q103.1 (G), R106.2
- new net: R115.2, R117.1
- new net: Q104.1 (G), R107.2
- new net: Q103.3 (D), R109.1
- new net: Q102.1 (G), R105.2
- new net: R116.2, R118.1
- new net: C116.1, FB101.2, U103.3 (VI)
- new net: R113.2, R114.1
- new net: Q104.3 (D), R110.1
- new net B_GATE: R107.1, U101.16 (GPIO10)
- new net B_OUT: J102.6 (Pin_6), R110.2
- new net CAN_RXD: U101.4 (XTAL_32K_P), U102.4 (R)
- new net CAN_TXD: U101.5 (XTAL_32K_N), U102.1 (D)
- new net EN: C120.1, D107.1 (K), R123.2, U101.7 (CHIP_EN)
- new net G_GATE: R106.1, U101.25 (GPIO18)
- new net G_OUT: J102.5 (Pin_5), R109.2
- new net JTRST: C123.1, D107.2 (A), J101.12 (~{RST})
- new net LNA_IN: C111.1, L102.1, U101.1 (LNA_IN)
- new net MTCK: D111.1 (K), J101.6 (JCLK/SWCLK), U101.12 (MTCK)
- new net MTDI: D110.1 (K), J101.10 (JTDI/NC), U101.10 (MTDI)
- new net MTDO: D112.1 (K), J101.8 (JTDO/SWO), U101.13 (MTDO)
- new net MTMS: D108.1 (K), J101.4 (JTMS/SWDIO), U101.9 (MTMS)
- new net NRZ1: R111.1, U101.8 (GPIO3)
- new net PI1_DIV: D101.2 (A), D108.2 (A), R103.2
- new net PI2_DIV: D104.2 (A), D110.2 (A), R114.2
- new net PI3_DIV: D105.2 (A), D112.2 (A), R117.2
- new net PI4_DIV: D106.2 (A), D111.2 (A), R118.2
- new net RF_ANT: AE101.2 (PCB_Trace), C112.1, L102.2
- new net R_GATE: R105.1, U101.15 (GPIO9)
- new net R_OUT: J102.16 (Pin_16), R108.2
- new net VCP_RX: J101.14 (VCP_TX), U101.27 (U0RXD)
- new net VCP_TX: J101.13 (VCP_RX), R122.2
- new net VDD: C103.1, C106.1, C107.1, C108.1, C109.1, C113.1, C114.1, C115.1, C117.1, D109.2 (A), L101.2, R123.1, R124.1, R125.1, U101.11 (VDD3P3_RTC), U101.17 (VDD3P3_CPU), U101.18 (VDD_SPI), U101.31 (VDDA), U101.32 (VDDA), U102.3 (VCC), U103.2 (VO)
- new net VS: C101.1, C102.1, FB101.1, J102.11 (Pin_11), Q101.3 (D)
- new net V_GATE: R104.1, U101.26 (GPIO19)
- new net V_OUT: J102.15 (Pin_15), R101.2
- new net XTAL_N: C105.1, U101.29 (XTAL_N), Y101.1
- new net XTAL_P: R121.2, U101.30 (XTAL_P)
- new net _VCP_TX: R122.1, U101.28 (U0TXD)
- new net _XTAL_P: C104.1, R121.1, Y101.3
- no-connect marks 2 -> 45
Other:
- removed sheet Application
- removed sheet BLE
- removed sheet CAN
- removed sheet Debugger
- removed sheet Digital Input
- removed sheet Power
- removed sheet RGB
- note removed: "3V3 TTL Input"
- note removed: "High Side Input"
- company: https://cone.codes -> (none)
- title: coneRGB2 -> (none)

Commit message: updates
Signed-off-by: Connor Rigby <connorr@hey.com>
Parts:
- added J104: FH34SRJ-6S-0.5SH(50), LCSC_Connector:FFC-SMD_6P-P0.50_FH34SRJ-6S-0.5SH, symbol Connector_Generic_MountingPin:Conn_01x06_MountingPin
- added SW101, SW104: TS-1101-C-W, Button:TS1101CW, symbol Switch:SW_Push
Connections:
- net GND: now also J104.1 (Pin_1)
- net MTCK: now also J104.6 (Pin_6), SW104.1
- net MTDI: now also J104.4 (Pin_4)
- net MTDO: now also J104.5 (Pin_5)
- net MTMS: now also J104.3 (Pin_3), SW101.1
- net VDD: now also J104.2 (Pin_2), SW101.2, SW104.2
- no-connect marks 45 -> 46

Commit message: updates
Parts:
- removed C110: C_0402_DNP, Capacitor_SMD:C_0402_1005Metric, symbol LCSC_Capacitor:C_0402_DNP
- removed C116, C117: C_0805_1u_X7R, Capacitor_SMD:C_0805_2012Metric, symbol LCSC_Capacitor:C_0805_1u_X7R
- removed U103: AMS1117-3.3, Package_TO_SOT_SMD:SOT-223-3_TabPin2, symbol Regulator_Linear:AMS1117-3.3
- added C1: 22uF, Capacitor_SMD:CP_Elec_4x5.4, symbol Device:C_Polarized_Small
- added C110: C_0402_100nf_X7R, Capacitor_SMD:C_0402_1005Metric, symbol LCSC_Capacitor:C_0402_100nf_X7R
- added C116, C3: 4.7uF, Capacitor_SMD:C_0805_2012Metric, symbol Device:C_Small
- added C117, C2: C_0805_10u_X5R, Capacitor_SMD:C_0805_2012Metric, symbol LCSC_Capacitor:C_0805_10u_X5R
- added TP1, TP2, TP3: TestPoint, TestPoint:TestPoint_Pad_D1.5mm, symbol Connector:TestPoint
- added TP4, TP5, TP6, TP7, TP8, TP9: TestPoint, TestPoint:TestPoint_Pad_D1.0mm, symbol Connector:TestPoint
- added U1: SPX3819M5-L-3-3/TR, Package_TO_SOT_SMD:SOT-23-5, symbol Regulator_Linear:SPX3819M5-L-3-3
- added U103: SPX1117M3-L-5-0/TR, Package_TO_SOT_SMD:SOT-223-3_TabPin2, symbol Regulator_Linear:AP1117-50
- C103, C106, C107, C108, C109, C113, C114, C115, C120, D101, D104, D105, D106, R102, R113, R115, R116, R119, R122, R123, R124, R125, Y101: now in the parts list
- C104, C105: Capacitance DNP -> 18pF; LCSC (none) -> C106202; now in the parts list
- C111, C112: Capacitance DNP -> 3.3pF; LCSC (none) -> C88892; now in the parts list
- FB101: value FerriteBead_Small -> 70mΩ ±25% 330Ω@100MH; LCSC (none) -> C74764
- H101, H102, H103, SW101, SW104: now not fitted; now left out of the parts list
- L101: value L_Small -> 2nH; LCSC (none) -> C142239
- L102: value L_Small -> 2.2nH; LCSC (none) -> C142238
- R101, R108, R109, R110: LCSC (none) -> C17408; now in the parts list
- R103, R114, R117, R118: LCSC (none) -> C21190; now in the parts list
- R104, R105, R106, R107: LCSC (none) -> C22775; now in the parts list
- R111: LCSC (none) -> C107696; now in the parts list
- R120: now not fitted
- R121: value R_0402_DNP -> 0R; LCSC (none) -> C17168; now in the parts list
Connections:
- net GND: now also C1.2, C110.2, C116.2, C117.2, C2.2, C3.2, TP3.1, U1.2 (GND), U103.1 (GND); no longer AE101.1 (FEED)
- net VDD: now also C117.1, TP2.1, U1.5 (OUT)
- net SPIHD: now reaches U101.19 (SPIHD)
- net SPIHD: now also TP4.1
- net at L101.1, U101.2 (VDD3P3), U101.3 (VDD3P3): now also C110.1
- net SPIWP: now reaches U101.20 (SPIWP)
- net SPIWP: now also TP5.1
- net SPICS0: now reaches U101.21 (SPICS0)
- net SPICS0: now also TP6.1
- net SPICLK: now reaches U101.22 (SPICLK)
- net SPICLK: now also TP7.1
- net SPID: now reaches U101.23 (SPID)
- net SPID: now also TP8.1
- net SPIQ: now reaches U101.24 (SPIQ)
- net SPIQ: now also TP9.1
- net at FB101.2: now also C1.1, C3.1, U103.3 (VI)
- new net +5V: C116.1, C2.1, TP1.1, U1.1 (IN), U1.3 (EN), U103.2 (VO)
- new net RF_STUB: AE101.1 (FEED)
- no-connect marks 46 -> 42
Other:
- moved on the sheet: AE101, FB101, L101, R123

Commit message: Prepare for Production
Parts:
- added H104: SMTSO2020CTJ, LCSC_Connector:SMTSO2020CTJ, symbol Mechanical:MountingHole_Pad
- AE101: MPN (none) -> C293767
- C101, C106, C113: LCSC C24123 -> C28323; MPN CL21B105KOFNNNE -> CL21B105KBFNNNE
- C102, C103, C109, C110, C114, C115, C120, C123: LCSC C110251 -> C1525; MPN 0402B104K500NT -> CL05B104KO5NNNC
- C104, C105: value C_0402_DNP -> C_0402_18p_NP0; LCSC C106202 -> C1549; MPN (none) -> 0402CG180J500NT
- C107: LCSC C1518210 -> C15195; MPN GRM1555CYA103JE01D -> CL05B103KB5NNNC
- C108, C117, C2: LCSC C162422 -> C15850; MPN GRM21BR6YA106KE43L -> CL21A106KAYNNNE
- C111, C112: value C_0402_DNP -> C_0402_3p3_C0G; LCSC C88892 -> C1565; MPN (none) -> 0402CG3R3C500NT
- C116, C3: LCSC C2857997 -> C1779; MPN (none) -> CL21A475KAQNNNE
- D102, D107, D108, D109, D110, D111, D112: LCSC C2927280 -> C191023; MPN (none) -> 1N5819WS
- FB101: value 70mΩ ±25% 330Ω@100MH -> 300mΩ ±25% 600Ω@100MHz; LCSC C74764 -> C1017; MPN (none) -> GZ2012D601TF
- H101, H102, H103: MPN (none) -> SMTSO2020CTJ
- J102: value ZE05H-16DP-2H -> ZE05H-16DP-2H; footprint LCSC_Connector:ZE05H-16DP-2H -> Harness:ZE05-16DS-HU; MPN (none) -> ZE05H-16DP-2H
- J103: footprint LCSC_Connector:ZE05H-16DP-2H -> Harness:ZE05-16DS-HU; MPN (none) -> ZE05-16DS-HU/R
- J104: MPN (none) -> FH34SRJ-6S-0.5SH(50)
- L101: MPN (none) -> CLH1005T-2N0S-S-NP
- L102: MPN (none) -> CLH1005T-2N2S-S-NP
- Q101: LCSC C306862 -> C15127; MPN (none) -> AO3401A
- Q102, Q103, Q104: LCSC C344010 -> C20917; MPN (none) -> AO3400A
- R101, R108, R109, R110: value 100 -> R_0805_100; MPN (none) -> 0805W8F1000T5E; Resistance (none) -> 100Ω
- R103, R114, R117, R118: value 1k -> R_0603_1k; MPN (none) -> 0603WAF1001T5E; Resistance (none) -> 1kΩ
- R104, R105, R106, R107: value 100 -> R_0603_100; MPN (none) -> 0603WAF1000T5E; Resistance (none) -> 100Ω
- R111: value 220 -> R_0603_220; LCSC C107696 -> C17557; MPN (none) -> 0805W8F2200T5E; Resistance (none) -> 220Ω
- R119, R123, R124, R125: LCSC C478866 -> C11702; MPN PTFR0402B1K00P9 -> 0402WGF1001TCE
- R121: value 0R -> R_0402_0; MPN (none) -> 0402WGF0000TCE; Resistance (none) -> 0Ω
- SW101, SW104: MPN (none) -> TS-1101-C-W
- T101, T102, T103, T104, T105, T106, T107, T108, T109, T110, T111, T112, T113, T114, T115, T116: value ZE05-2022SCF -> ZE05-2022SCF; footprint (none) -> Harness:ZE05-2022SCF; MPN (none) -> ZE05-2022SCF
- U1: MPN (none) -> SPX3819M5-L-3-3/TR
- U101: MPN (none) -> ESP32-C3FH4
- U102: MPN (none) -> SN65HVD230DR
- U103: LCSC C21946 -> C6187; MPN (none) -> SPX1117M3-L-5-0/TR
Connections:
- no-connect marks 42 -> 43

Commit message: submit for production
Signed-off-by: Connor Rigby <connorr@hey.com>
Parts:
- H101, H102, H103, H104: value SMTSO2020CTJ -> MountingHole; footprint LCSC_Connector:SMTSO2020CTJ -> MountingHole:MountingHole_2.2mm_M2_Pad_Via; LCSC C2915626 -> (none); MPN SMTSO2020CTJ -> (none); now fitted
- J101: TAG_CONNECT (none) -> https://www.tag-connect.com/wp-content/uploads/bsk-pdf-mana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
Connections:
- net GND: now also H101.1, H102.1, H103.1, H104.1
- no-connect marks 43 -> 39
